Commit message: update double pendulum

File: double_pendulum.urdf (robot description, URDF)
Before this commit: robot pendulum, 6 links, 5 joints
Joints:
- joint joint_1: axis 0 1 0 -> 0 -1 0; origin xyz=0.0 0 0 rpy=0 3.14159265 0 -> xyz=0.0 0 0 rpy=0 3.14159265358979323846 0
- joint joint_2: origin xyz=0.0 0 0 rpy=0 3.14159265 0 -> xyz=0.0 0 0 rpy=0 0 0
